File: nest_interface/eagle/rev_a/nest_interface_a.brd (EAGLE design)
At the start: 114.3 x 83.8 mm, 175 parts, among them J1 MOLEX_MICRO_USB_B_047346, J10 CONN_BLOCK_2, J11 CONN_BLOCK_2, J12 CONN_BLOCK_2, J13 CONN_BLOCK_2, J14 CONN_BLOCK_2, J15 CONN_BLOCK_2, J16 CONN_BLOCK_3, J17 CONN_BLOCK_3, J18 CONN_BLOCK_2, J19 CONN_BLOCK_3, J2 CONN_BLOCK_2, J20 CONN_BLOCK_3, J21 CONN_BLOCK_3, J22 CONN_BLOCK_2, J23 CONN_BLOCK_3, J24 CONN_BLOCK_3, J25 MOLEX_MICRO_USB_B_047346, J3 CONN_BLOCK_3, J4 PJ-036A-SMT, J5 CONN_BLOCK_3, J6 CONN_BLOCK_3, J7 CONN_BLOCK_2, J8 CONN_BLOCK_3, J9 CONN_BLOCK_3, U1 FT232RL, U2 EPIC-CORE_A, U3 MPC1825, U4 PCA9575, U5 PCA9575, U6 FT232RL, Y1 FC-135_32.768KA-A3

Commit message: started routing wow is that going to be tricky
Parts:
- removed J10, J18, J22: CONN_BLOCK_2, nest_interface:CONN_BLOCK_2
- removed J16, J19, J20, J21, J9: CONN_BLOCK_3, nest_interface:CONN_BLOCK_3
- removed Q1, Q10, Q11, Q12, Q13, Q14, Q2, Q3, Q4, Q5, Q6, Q7, Q8, Q9: (no value), nest_interface:SOT23-3
- removed R12, R14, R16, R18, R20, R22, R24, R26, R28, R30, R32, R34, R36, R40, R41, R42, R43, R44, R45, R46, R47, R48, R49, R50, R51, R52, R53, R54, R55, R56, R57, R58, R59, R60, R61, R62, R63, R64, R65, R68, R69: 100k, rcl:R0603
- removed R13, R15, R17, R19, R21, R23, R25, R27, R29, R31, R70, R71: 10k, rcl:R0603
- removed RA3: VSSR2403103, nest_interface:LSSOP-24
- removed U$1, U$2, U$3, U$4: ALD1107, nest_interface:SOIC-14
- removed U$5: MSP430F1611IPM, hijack:PM/PAG64
- added J30: PINH2X12, SparkFun:2X12
- added QA1, QA2, QA3, QA4: MMPQ2222A, nest_interface:SOIC-16
- added RA5, RA6: 766161104GP, nest_interface:SOIC-16
- added RA7: VSSR1603103, nest_interface:LSSOP-16
- added U10, U11, U8, U9: ALD1107, nest_interface:SOIC-14
- added U20: MSP430F1611IPM, hijack:PM/PAG64
- added U7: TC1262, nest_interface:SOT-223-3
- J23, J24, J5, J6: value CONN_BLOCK_3 -> CONN_BLOCK_8; device nest_interface:CONN_BLOCK_3 -> nest_interface:CONN_BLOCK_8
- J7: value CONN_BLOCK_2 -> CONN_BLOCK_7; device nest_interface:CONN_BLOCK_2 -> nest_interface:CONN_BLOCK_7
- J8: value CONN_BLOCK_3 -> CONN_BLOCK_7; device nest_interface:CONN_BLOCK_3 -> nest_interface:CONN_BLOCK_7
- R10: value 100k -> 10k
- R66, R67: value 0 -> 100k
- R9: value 10k -> 100k
- moved D10 457.1 mm to (69.3, 86.6)
- moved RA4 454.7 mm to (162.6, 64.8), turned to 180 degrees
- moved R80 452.4 mm to (67.3, 86.6), turned to 90 degrees
- moved D9 451.6 mm to (73.7, 86.6)
- moved R79 446.9 mm to (71.6, 86.6), turned to 90 degrees
- moved R78 443.8 mm to (75.9, 86.6), turned to 90 degrees
- moved D8 440.3 mm to (78.0, 86.6)
- moved RA2 421.5 mm to (74.4, 97.0), turned to 180 degrees
- moved RA1 400.5 mm to (84.6, 97.0)
- moved C17 392.1 mm to (72.4, 116.8)
- moved R77 385.9 mm to (68.6, 116.8)
- moved J24 381.3 mm to (212.1, 99.1), turned to 90 degrees
- moved C16 372.9 mm to (62.2, 115.6)
- moved R75 366.7 mm to (58.4, 115.6)
- moved Y1 358.5 mm to (53.3, 115.6)
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Connections:
- net MISO0 renamed EPIC_MISO0
- net P2.0 renamed EPIC_P2.0
- net P2.4 renamed EPIC_P2.4
- net P2.7 renamed EPIC_P2.7
- net STE0 renamed EPIC_STE0
- net UART0RX renamed EPIC_UART0RX
- net UART0TX renamed EPIC_UART0TX
- removed net ADC5: JP1.16, U2.P$24
- removed net ADC6/DAC0: JP1.14, U2.P$25
- removed net ADC7/DAC1: JP1.12, U2.P$26
- removed net MOSI0/SDA: JP1.11
- removed net N$16: Q2.1, R11.1
- removed net N$17: Q1.1, R9.1
- removed net N$25: Q3.1, R13.1
- removed net N$26: Q4.1, R15.1
- removed net N$27: Q5.1, R17.1
- removed net N$28: Q6.1, R19.1
- removed net N$29: Q7.1, R21.1
- removed net N$30: Q8.1, R23.1
- removed net N$31: Q9.1, R25.1
- removed net N$32: Q10.1, R27.1
- removed net N$33: Q11.1, R29.1
- removed net N$34: Q12.1, R31.1
- removed net N$42: J25.ID, L2.1
- removed net N$5: J1.ID, L1.1
- removed net SCLK0/SCL: JP1.15
- removed net TSTAT1_DOWN: J6.1
- removed net TSTAT1_ENTER: J7.2
- removed net TSTAT1_ESC: J6.3
- removed net TSTAT1_HELP: J6.2
- removed net TSTAT1_LCD_DB0: J19.1, RA1.7
- removed net TSTAT1_LCD_DB0_PIN: RA1.17, RA1.18, U$5.36
- removed net TSTAT1_LCD_DB1: J19.2, RA1.9
- removed net TSTAT1_LCD_DB1_PIN: RA1.15, RA1.16, U$5.37
- removed net TSTAT1_LCD_DB2: J19.3, RA1.11
- removed net TSTAT1_LCD_DB2_PIN: RA1.13, RA1.14, U$5.38
- removed net TSTAT1_LCD_DB3: J20.1, RA2.1
- removed net TSTAT1_LCD_DB3_PIN: RA2.23, RA2.24, U$5.39
- removed net TSTAT1_MENU: J5.2
- removed net TSTAT1_ON/OFF: J5.3
- removed net TSTAT1_UP: J5.1
- removed net TSTAT2_DOWN: J9.1
- removed net TSTAT2_ENTER: J10.2
- removed net TSTAT2_ESC: J9.3
- removed net TSTAT2_HELP: J9.2
- removed net TSTAT2_LCD_DB0: J23.1, RA3.7
- removed net TSTAT2_LCD_DB0_PIN: RA3.17, RA3.18, U$5.59
- removed net TSTAT2_LCD_DB1: J23.2, RA3.9
- removed net TSTAT2_LCD_DB1_PIN: RA3.15, RA3.16, U$5.60
- removed net TSTAT2_LCD_DB2: J23.3, RA3.11
- removed net TSTAT2_LCD_DB2_PIN: RA3.13, RA3.14, U$5.61
- removed net TSTAT2_LCD_DB3: J24.1, RA4.1
- removed net TSTAT2_LCD_DB3_PIN: RA4.23, RA4.24, U$5.2
- removed net TSTAT2_MENU: J8.2
- removed net TSTAT2_ON/OFF: J8.3
- removed net TSTAT2_UP: J8.1
- new net 5.6V_SUPPLY: J11.2, U3.1, U7.1
- new net EPIC_ADC1: JP1.18, U2.P$20
- new net EPIC_ADC2: JP1.16, U2.P$21
- new net EPIC_ADC3: JP1.14, U2.P$22
- new net EPIC_ADC4: JP1.12, U2.P$23
- new net EPIC_ADC5: JP1.10, U2.P$24
- new net EPIC_ADC6/DAC0: JP1.8, U2.P$25
- new net EPIC_ADC7/DAC1: JP1.6, U2.P$26
- new net EPIC_P5.7: JP1.7, U2.P$9
- new net LCDP_MISO0: J30.16, U20.30
- new net LCDP_P2.4: J30.4, U20.24
- new net LCDP_P2.7: U20.27
- new net LCDP_STE0: J30.18, U20.28
- new net LCDP_URXD0: J30.12, U20.33
- new net LCDP_UTXD0: J30.14, U20.32
- new net N$59: QA1.11, RA4.22
- new net N$60: QA1.9, RA4.21
- new net N$61: QA2.15, RA4.20
- new net N$62: QA2.13, RA4.19
- new net N$63: QA2.11, RA4.18
- new net N$64: QA2.9, RA4.17
- new net N$65: QA3.15, RA4.16
- new net N$66: QA3.13, RA4.15
- new net N$67: QA3.11, RA4.14
- new net N$68: QA3.9, RA4.13
- new net P1.6: J30.10, U20.18
- new net P1.7: J30.8, U20.19
- new net P2.3: J30.6, U20.23
- new net P2.6: J30.2, U20.26
- new net P5.0: J30.1, U20.44
- new net P5.1: J30.3, U20.45
- new net P5.2: J30.5, U20.46
- new net P5.3: J30.7, U20.47
- new net P5.4: J30.9, U20.48
- new net P5.5: U20.49
- new net P5.6: J30.11, U20.50
- new net P5.7: J30.13, U20.51
- new net P6.0: J30.15, U20.59
- new net P6.1: J30.17, U20.60
- new net P6.2: J30.19, U20.61
- new net P6.3: J30.21, U20.2
- new net P6.4: J30.23, U20.3
- new net P6.5: J30.24, U20.4
- new net P6.6: J30.22, U20.5
- new net P6.7: J30.20, U20.6
- new net TSTAT_IN_I2C_RST: R66.2, U2.P$2, U4.3
- new net TSTAT_OUT_I2C_RST: R67.2, U2.P$3, U5.3
- net #KEYPAD_ENABLE: now also R9.1, U10.13, U10.2, U10.6, U10.9, U11.13, U11.2, U2.P$4, U8.13, U8.2, U8.6, U8.9, U9.13, U9.2, U9.6, U9.9; no longer R40.2, R41.2, R42.2, R43.2, R48.2, R49.2, R50.2, R51.2, R56.2, R57.2, R58.2, R59.2, R64.2, R65.2, U$1.13, U$1.2, U$1.6, U$1.9, U$2.13, U$2.2, U$2.6, U$2.9, U$3.13, U$3.2, U$3.6, U$3.9, U$4.13, U$4.2
- net 5V: now also U7.3; no longer J11.2, U3.1
- net GND: now also J23.1, J24.1, J5.1, J6.1, QA1.10, QA1.12, QA1.14, QA1.16, QA2.10, QA2.12, QA2.14, QA2.16, QA3.10, QA3.12, QA3.14, QA3.16, QA4.14, QA4.16, R9.2, RA2.12, RA5.16, RA7.2, RA7.4, U10.4, U11.4, U20.10, U20.11, U20.53, U20.62, U20.63, U7.2, U7.4, U8.4, U9.4; no longer J10.1, J7.1, Q1.2, Q10.2, Q11.2, Q12.2, Q13.2, Q14.2, Q2.2, Q3.2, Q4.2, Q5.2, Q6.2, Q7.2, Q8.2, Q9.2, R10.2, R12.2, R14.2, R16.2, R18.2, R20.2, R22.2, R24.2, R26.2, R28.2, R30.2, R32.2, R34.2, R36.2, R40.1, R41.1, R42.1, R43.1, R48.1, R49.1, R50.1, R51.1, R56.1, R57.1, R58.1, R59.1, R64.1, R65.1, RA3.10, RA3.12, RA3.2, RA3.4, RA3.6, RA3.8, RA4.10, RA4.2, RA4.4, RA4.6, RA4.8, U$1.4, U$2.4, U$3.4, U$4.4, U$5.10, U$5.11, U$5.53, U$5.62, U$5.63
- net I2C_SCL: now also JP1.15, R10.2, U20.31; no longer R70.1, U$5.31
- net I2C_SDA: now also JP1.11, R11.2, U20.29; no longer R71.1, U$5.29
- net N$1: now also L1.1
- net N$35: no longer Q13.1
- net N$36: no longer Q14.1
- net N$37: now also QA1.15, RA4.24; no longer R66.2, U4.3
- net N$38: now also U20.8; no longer U$5.8
- net N$39: now also L2.1
- net N$48: now also U20.34; no longer U$5.34
- net N$49: now also U20.35
- net N$50: now also U20.57; no longer U$5.57
- net N$52: now also U20.9; no longer U$5.9
- net N$54: now also U20.25; no longer U$5.25
- net N$56: now also U20.21; no longer U$5.21
- net N$57: now also U20.22; no longer U$5.22
- net N$58: now also QA1.13, RA4.23; no longer R67.2, U5.3
- net N$8: now also U20.20; no longer U$5.20
- net RADIO_SFD: now also JP1.4; no longer JP1.10
- net RST1: now also U20.58; no longer U$5.58
- net TSTAT1_DOWN_IN: now also J5.3, RA6.6, U4.5, U9.12; no longer R53.1, U$2.12, U4.11
- net TSTAT1_DOWN_OUT: now also J23.3, QA2.3, QA2.4, U9.14; no longer Q6.3, U$2.14
- net TSTAT1_DOWN_OUT_PIN: now also RA4.6, RA5.3; no longer R19.2, R20.1
- net TSTAT1_ENTER_IN: now also J5.2, RA6.7, U4.4, U9.8; no longer R54.1, U$2.8, U4.12
- net TSTAT1_ENTER_OUT: now also J23.2, QA2.5, QA2.6, U9.10; no longer Q7.3, U$2.10
- net TSTAT1_ENTER_OUT_PIN: now also RA4.7, RA5.2; no longer R21.2, R22.1
- net TSTAT1_ESC_IN: now also J5.5, RA6.4, U8.7; no longer R47.1, U$1.7
- net TSTAT1_ESC_OUT: now also J23.5, QA1.7, QA1.8, U8.5; no longer Q4.3, U$1.5
- net TSTAT1_ESC_OUT_PIN: now also RA4.4, RA5.5; no longer R15.2, R16.1
- net TSTAT1_HELP_IN: now also J5.4, RA6.5, U4.6, U9.3; no longer R52.1, U$2.3, U4.10
- net TSTAT1_HELP_OUT: now also J23.4, QA2.1, QA2.2, U9.1; no longer Q5.3, U$2.1
- net TSTAT1_HELP_OUT_PIN: now also RA4.5, RA5.4; no longer R17.2, R18.1
- net TSTAT1_LCD_DB4: now also J7.4, RA1.7; no longer J20.2, RA2.3
- net TSTAT1_LCD_DB4_PIN: now also RA1.17, RA1.18, U20.36; no longer RA2.21, RA2.22, U$5.40
- net TSTAT1_LCD_DB5: now also J7.5, RA1.9; no longer J20.3, RA2.5
- net TSTAT1_LCD_DB5_PIN: now also RA1.15, RA1.16, U20.37; no longer RA2.19, RA2.20, U$5.41
- net TSTAT1_LCD_DB6: now also J7.6, RA1.11; no longer J18.1, RA2.7
- net TSTAT1_LCD_DB6_PIN: now also RA1.13, RA1.14, U20.38; no longer RA2.17, RA2.18, U$5.42
- net TSTAT1_LCD_DB7: now also J7.7, RA2.1; no longer J18.2, RA2.9
- net TSTAT1_LCD_DB7_PIN: now also RA2.23, RA2.24, U20.39; no longer RA2.15, RA2.16, U$5.43
- net TSTAT1_LCD_E: now also J7.3; no longer J16.3
- net TSTAT1_LCD_E_PIN: now also U20.15; no longer U$5.14
- net TSTAT1_LCD_R/W: now also J7.2; no longer J16.2
- net TSTAT1_LCD_R/W_PIN: now also U20.16; no longer U$5.13
- net TSTAT1_LCD_RS: now also J7.1; no longer J16.1
- net TSTAT1_LCD_RS_PIN: now also U20.17; no longer U$5.12
- net TSTAT1_MENU_IN: now also J5.7, RA6.2, U4.11, U8.12; no longer R45.1, U$1.12, U4.5
- net TSTAT1_MENU_OUT: now also J23.7, QA1.3, QA1.4, U8.14; no longer Q2.3, U$1.14
- net TSTAT1_MENU_OUT_PIN: now also RA4.2, RA5.7; no longer R11.2, R12.1
- net TSTAT1_ON/OFF_IN: now also J5.8, RA6.1, U4.12, U8.3; no longer R44.1, U$1.3, U4.4
- net TSTAT1_ON/OFF_OUT: now also J23.8, QA1.1, QA1.2, U8.1; no longer Q1.3, U$1.1
- net TSTAT1_ON/OFF_OUT_PIN: now also RA4.1, RA5.8; no longer R10.1, R9.2
- net TSTAT1_UP_IN: now also J5.6, RA6.3, U4.10, U8.8; no longer R46.1, U$1.8, U4.6
- net TSTAT1_UP_OUT: now also J23.6, QA1.5, QA1.6, U8.10; no longer Q3.3, U$1.10
- net TSTAT1_UP_OUT_PIN: now also RA4.3, RA5.6; no longer R13.2, R14.1
- net TSTAT2_DOWN_IN: now also J6.3, RA6.13, U11.3; no longer R68.1, U$4.3
- net TSTAT2_DOWN_OUT: now also J24.3, QA4.1, QA4.2, U11.1; no longer Q13.3, U$4.1
- net TSTAT2_DOWN_OUT_PIN: now also RA5.13; no longer R34.1
- net TSTAT2_ENTER_IN: now also J6.2, RA6.14, U11.12; no longer R69.1, U$4.12
- net TSTAT2_ENTER_OUT: now also J24.2, QA4.3, QA4.4, U11.14; no longer Q14.3, U$4.14
- net TSTAT2_ENTER_OUT_PIN: now also RA5.14; no longer R36.1
- net TSTAT2_ESC_IN: now also J6.5, RA6.11, U10.8; no longer R62.1, U$3.8
- net TSTAT2_ESC_OUT: now also J24.5, QA3.5, QA3.6, U10.10; no longer Q11.3, U$3.10
- net TSTAT2_ESC_OUT_PIN: now also RA4.11, RA5.10; no longer R29.2, R30.1
- net TSTAT2_HELP_IN: now also J6.4, RA6.12, U10.7; no longer R63.1, U$3.7
- net TSTAT2_HELP_OUT: now also J24.4, QA3.7, QA3.8, U10.5; no longer Q12.3, U$3.5
- net TSTAT2_HELP_OUT_PIN: now also RA4.12, RA5.9; no longer R31.2, R32.1
- net TSTAT2_LCD_DB4: now also J8.4, RA2.9; no longer J24.2, RA4.3
- net TSTAT2_LCD_DB4_PIN: now also RA2.15, RA2.16, U20.40; no longer RA4.21, RA4.22, U$5.3
- net TSTAT2_LCD_DB5: now also J8.5, RA2.11; no longer J24.3, RA4.5
- net TSTAT2_LCD_DB5_PIN: now also RA2.13, RA2.14, U20.41; no longer RA4.19, RA4.20, U$5.4
- net TSTAT2_LCD_DB6: now also J8.6, RA7.1; no longer J22.1, RA4.7
- net TSTAT2_LCD_DB6_PIN: now also RA7.15, RA7.16, U20.42; no longer RA4.17, RA4.18, U$5.5
- net TSTAT2_LCD_DB7: now also J8.7, RA7.3; no longer J22.2, RA4.9
- net TSTAT2_LCD_DB7_PIN: now also RA7.13, RA7.14, U20.43; no longer RA4.15, RA4.16, U$5.6
- net TSTAT2_LCD_E: now also J8.3, RA2.7; no longer J21.3, RA3.5
- net TSTAT2_LCD_E_PIN: now also RA2.17, RA2.18, U20.14; no longer RA3.19, RA3.20, U$5.17
- net TSTAT2_LCD_R/W: now also J8.2, RA2.5; no longer J21.2, RA3.3
- net TSTAT2_LCD_R/W_PIN: now also RA2.19, RA2.20, U20.13; no longer RA3.21, RA3.22, U$5.16
- net TSTAT2_LCD_RS: now also J8.1, RA2.3; no longer J21.1, RA3.1
- net TSTAT2_LCD_RS_PIN: now also RA2.21, RA2.22, U20.12; no longer RA3.23, RA3.24, U$5.15
- net TSTAT2_MENU_IN: now also J6.7, RA6.9, U10.3; no longer R60.1, U$3.3
- net TSTAT2_MENU_OUT: now also J24.7, QA3.1, QA3.2, U10.1; no longer Q9.3, U$3.1
- net TSTAT2_MENU_OUT_PIN: now also RA4.9, RA5.12; no longer R25.2, R26.1
- net TSTAT2_ON/OFF_IN: now also J6.8, RA6.8, U9.7; no longer R55.1, U$2.7
- net TSTAT2_ON/OFF_OUT: now also J24.8, QA2.7, QA2.8, U9.5; no longer Q8.3, U$2.5
- net TSTAT2_ON/OFF_OUT_PIN: now also RA4.8, RA5.1; no longer R23.2, R24.1
- net TSTAT2_UP_IN: now also J6.6, RA6.10, U10.12; no longer R61.1, U$3.12
- net TSTAT2_UP_OUT: now also J24.6, QA3.3, QA3.4, U10.14; no longer Q10.3, U$3.14
- net TSTAT2_UP_OUT_PIN: now also RA4.10, RA5.11; no longer R27.2, R28.1
- net TSTAT_IN_I2C_INT: now also U2.P$30
- net VCC: now also R10.1, R11.1, RA6.16, U10.11, U11.11, U20.1, U20.64, U8.11, U9.11; no longer R44.2, R45.2, R46.2, R47.2, R52.2, R53.2, R54.2, R55.2, R60.2, R61.2, R62.2, R63.2, R68.2, R69.2, R70.2, R71.2, U$1.11, U$2.11, U$3.11, U$4.11, U$5.1, U$5.64
Routing:
- net COMMON: track 129.2 -> 32.0 mm
- net VCC: track 273.6 -> 222.2 mm
- net TSTAT2_HELP_OUT_PIN: track 2.79 -> 48.7 mm, vias 0 -> 2
- net TSTAT2_ESC_OUT_PIN: track 2.79 -> 48.0 mm, vias 0 -> 2
- net TSTAT2_UP_OUT_PIN: track 2.79 -> 46.6 mm, vias 0 -> 2
- net TSTAT1_LCD_RS_PIN: track 0.00 -> 43.4 mm, vias 0 -> 2
- net TSTAT1_LCD_R/W_PIN: track 0.00 -> 42.9 mm, vias 0 -> 2
- net TSTAT2_MENU_OUT_PIN: track 2.79 -> 44.9 mm, vias 0 -> 2
- net TSTAT1_LCD_E_PIN: track 0.00 -> 41.2 mm, vias 0 -> 2
- net 5V: track 50.3 -> 13.5 mm
- net SCLK0/SCL: track 34.2 -> 0.00 mm, vias 1 -> 0
- net I2C_SCL: track 0.00 -> 34.2 mm, vias 0 -> 1
- net TSTAT2_LCD_RS_PIN: track 0.00 -> 33.7 mm, vias 0 -> 2
- net MOSI0/SDA: track 33.1 -> 0.00 mm, vias 1 -> 0
- net I2C_SDA: track 0.00 -> 33.1 mm, vias 0 -> 1
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- added copper zone on layer 1, net COMMON
- added copper zone on layer 1, net RH
Other:
- board size 114.3 x 83.8 mm -> 105.4 x 110.5 mm
- board text added: "DB4"
- board text added: "DB5"
- board text added: "DB6"
- board text added: "DB7"
- board text added: "E"
- board text added: "R/W"
- board text added: "RS"
- board text removed: "3V"

Commit message: cleaning up schematic/bom
Parts:
- removed R37, R38, R39: 100k, rcl:R0603
- added R101, R102: 10k, rcl:R0603
- added R99: 100k, rcl:R0603
- C10, C11, C6, C7, C8, C9: value (none) -> .1u
- R10, R11: value 10k -> 100k
- moved R9 76.2 mm to (45.5, 9.14), turned to 180 degrees
- moved R10 75.3 mm to (45.5, 22.6), turned to 180 degrees
- moved R11 68.1 mm to (45.5, 35.3), turned to 180 degrees
- moved C10 39.6 mm to (45.5, 25.9)
- moved C11 39.6 mm to (45.5, 39.1)
- moved C6 39.6 mm to (45.5, 52.3)
- moved C7 39.6 mm to (45.5, 65.5)
- moved C8 39.6 mm to (45.5, 78.7)
- moved C9 39.6 mm to (45.5, 12.7)
Connections:
- net #KEYPAD_ENABLE: now also R99.1; no longer R9.1
- net COOLING1_PIN: now also C7.1; no longer C10.1
- net COOLING2_PIN: now also C10.1, R10.1; no longer C7.1, R38.1
- net FAN_PIN: now also C8.1; no longer C11.1
- net GND: now also R99.2; no longer R9.2
- net HEATING1_PIN: now also C6.1; no longer C9.1
- net HEATING2_PIN: now also C9.1, R9.1; no longer C6.1, R37.1
- net I2C_SCL: now also R101.2; no longer R10.2
- net I2C_SDA: now also R102.2; no longer R11.2
- net STAR_PIN: now also C11.1, R11.1; no longer C8.1, R39.1
- net VCC: now also R10.2, R101.1, R102.1, R11.2, R9.2; no longer R10.1, R11.1, R37.2, R38.2, R39.2

Commit message: routing
Parts:
- removed QA4: MMPQ2222A, nest_interface:SOIC-16
- added Q1, Q2: (no value), nest_interface:SOT23
- moved J24 143.8 mm to (123.2, -14.0)
- moved R35 110.2 mm to (167.1, 86.6), turned to 270 degrees
- moved R33 109.1 mm to (169.4, 86.6), turned to 270 degrees
- moved J23 106.5 mm to (157.5, -15.2), turned to 180 degrees
- moved U11 86.7 mm to (168.1, 94.0), turned to 90 degrees
- moved U9 42.0 mm to (182.6, 56.1), turned to 270 degrees
- moved RA6 35.9 mm to (204.2, 49.5), turned to 180 degrees
- moved U10 34.0 mm to (159.8, 45.7), turned to 180 degrees
- moved U8 33.1 mm to (182.6, 67.1), turned to 270 degrees
- moved QA1 16.3 mm to (172.5, 67.1), turned to 180 degrees
- moved QA2 13.3 mm to (171.2, 55.4)
- moved QA3 13.3 mm to (159.8, 55.4)
- moved RA4 3.59 mm to (160.0, 67.3)
Connections:
- removed net N$35: R33.1
- removed net N$36: R35.1
- removed net N$59: QA1.11, RA4.22
- removed net N$61: QA2.15, RA4.20
- removed net N$62: QA2.13, RA4.19
- removed net N$63: QA2.11, RA4.18
- removed net N$64: QA2.9, RA4.17
- removed net N$66: QA3.13, RA4.15
- removed net N$67: QA3.11, RA4.14
- removed net N$68: QA3.9, RA4.13
- new net N$16: QA1.11, RA4.23
- new net N$17: QA2.13, RA4.18
- new net N$25: QA2.11, RA4.19
- new net N$26: QA2.9, RA4.20
- new net N$28: QA3.15, RA4.13
- new net N$29: QA3.13, RA4.14
- new net N$30: QA3.11, RA4.15
- new net N$31: Q1.1, R33.1
- new net N$32: Q2.1, R35.1
- new net N$5: QA2.15, RA4.17
- net GND: now also Q1.2, Q2.2; no longer QA4.14, QA4.16
- net N$37: now also QA1.9; no longer QA1.15
- net N$58: now also RA4.22; no longer RA4.23
- net N$60: now also QA1.15; no longer QA1.9
- net N$65: now also QA3.9; no longer QA3.15
- net TSTAT1_DOWN_IN: now also RA6.3; no longer RA6.6
- net TSTAT1_DOWN_OUT: now also QA2.5, QA2.6; no longer QA2.3, QA2.4
- net TSTAT1_ENTER_IN: now also RA6.2; no longer RA6.7
- net TSTAT1_ENTER_OUT: now also QA2.3, QA2.4; no longer QA2.5, QA2.6
- net TSTAT1_ESC_IN: now also RA6.5; no longer RA6.4
- net TSTAT1_ESC_OUT: now also QA1.1, QA1.2; no longer QA1.7, QA1.8
- net TSTAT1_HELP_IN: now also RA6.4; no longer RA6.5
- net TSTAT1_HELP_OUT: now also QA2.7, QA2.8; no longer QA2.1, QA2.2
- net TSTAT1_MENU_IN: now also RA6.7; no longer RA6.2
- net TSTAT1_MENU_OUT: now also QA1.5, QA1.6; no longer QA1.3, QA1.4
- net TSTAT1_ON/OFF_IN: now also RA6.8; no longer RA6.1
- net TSTAT1_ON/OFF_OUT: now also QA1.7, QA1.8; no longer QA1.1, QA1.2
- net TSTAT1_UP_IN: now also RA6.6; no longer RA6.3
- net TSTAT1_UP_OUT: now also QA1.3, QA1.4; no longer QA1.5, QA1.6
- net TSTAT2_DOWN_IN: now also RA6.14; no longer RA6.13
- net TSTAT2_DOWN_OUT: now also Q1.3; no longer QA4.1, QA4.2
- net TSTAT2_ENTER_IN: now also RA6.15; no longer RA6.14
- net TSTAT2_ENTER_OUT: now also Q2.3; no longer QA4.3, QA4.4
- net TSTAT2_ESC_IN: now also RA6.12; no longer RA6.11
- net TSTAT2_ESC_OUT: now also QA3.3, QA3.4; no longer QA3.5, QA3.6
- net TSTAT2_ESC_OUT_PIN: now also RA5.11; no longer RA5.10
- net TSTAT2_HELP_IN: now also RA6.13; no longer RA6.12
- net TSTAT2_HELP_OUT: now also QA3.1, QA3.2; no longer QA3.7, QA3.8
- net TSTAT2_HELP_OUT_PIN: now also RA5.12; no longer RA5.9
- net TSTAT2_MENU_IN: now also RA6.10; no longer RA6.9
- net TSTAT2_MENU_OUT: now also QA3.7, QA3.8; no longer QA3.1, QA3.2
- net TSTAT2_MENU_OUT_PIN: now also RA5.9; no longer RA5.12
- net TSTAT2_ON/OFF_IN: now also RA6.9; no longer RA6.8
- net TSTAT2_ON/OFF_OUT: now also QA2.1, QA2.2; no longer QA2.7, QA2.8
- net TSTAT2_UP_IN: now also RA6.11; no longer RA6.10
- net TSTAT2_UP_OUT: now also QA3.5, QA3.6; no longer QA3.3, QA3.4
- net TSTAT2_UP_OUT_PIN: now also RA5.10; no longer RA5.11
Routing:
- net #KEYPAD_ENABLE: track 0.00 -> 60.7 mm
- net GND: track 102.0 -> 148.3 mm, vias 22 -> 29
- net TSTAT2_HELP_IN: track 16.1 -> 54.1 mm, vias 0 -> 1
- net TSTAT2_ESC_IN: track 13.1 -> 49.8 mm, vias 0 -> 1
- net TSTAT2_UP_IN: track 11.3 -> 46.4 mm, vias 0 -> 1
- net TSTAT2_MENU_IN: track 9.51 -> 43.1 mm, vias 0 -> 1
- net TSTAT2_ON/OFF_IN: track 9.01 -> 41.3 mm, vias 0 -> 1
- net TSTAT2_ENTER_IN: track 21.0 -> 48.6 mm
- net TSTAT2_DOWN_IN: track 18.2 -> 43.5 mm
- net TSTAT2_ENTER_OUT_PIN: track 0.00 -> 23.6 mm
- net TSTAT1_DOWN_OUT: track 0.00 -> 22.6 mm
- net TSTAT1_ENTER_OUT: track 0.00 -> 22.3 mm
- net TSTAT2_DOWN_OUT_PIN: track 0.00 -> 20.1 mm
- net N$26: track 0.00 -> 19.5 mm
- net TSTAT2_ON/OFF_OUT: track 0.00 -> 19.1 mm
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