File: nest_interface/eagle/rev_a/nest_interface_a.sch (EAGLE design)
At the start: 108 parts, among them J1 MOLEX_MICRO_USB_B_047346, J11 CONN_BLOCK_2, J12 CONN_BLOCK_2, J13 CONN_BLOCK_2, J14 CONN_BLOCK_2, J15 CONN_BLOCK_2, J17 CONN_BLOCK_3, J2 CONN_BLOCK_2, J23 CONN_BLOCK_8, J24 CONN_BLOCK_8, J25 MOLEX_MICRO_USB_B_047346, J3 CONN_BLOCK_3, J30 PINH2X12, J4 PJ-036A-SMT, J5 CONN_BLOCK_8, J6 CONN_BLOCK_8, J7 CONN_BLOCK_7, J8 CONN_BLOCK_7, U1 FT232RL, U10 ALD1107, U11 ALD1107, U2 EPIC-CORE_A, U20 MSP430F1611IPM, U3 MPC1825, U4 PCA9575, U5 PCA9575, U6 FT232RL, U7 TC1262, U8 ALD1107, U9 ALD1107, Y1 FC-135_32.768KA-A3

Commit message: cleaning up schematic/bom
Parts:
- removed R37, R38, R39: 100k, rcl:R-US_R0603
- added R101, R102: 10k, rcl:R-US_R0603
- added R99: 100k, rcl:R-US_R0603
- C10, C11, C6, C7, C8, C9: value (none) -> .1u
- R10, R11: value 10k -> 100k
Connections:
- net #KEYPAD_ENABLE: now also R99.1; no longer R9.1
- net COOLING1_PIN: now also C7.1; no longer C10.1
- net COOLING2_PIN: now also C10.1, R10.1; no longer C7.1, R38.1
- net FAN_PIN: now also C8.1; no longer C11.1
- net GND: now also R99.2; no longer R9.2
- net HEATING1_PIN: now also C6.1; no longer C9.1
- net HEATING2_PIN: now also C9.1, R9.1; no longer C6.1, R37.1
- net I2C_SCL: now also R101.2; no longer R10.2
- net I2C_SDA: now also R102.2; no longer R11.2
- net STAR_PIN: now also C11.1, R11.1; no longer C8.1, R39.1
- net VCC: now also R10.2, R101.1, R102.1, R11.2, R9.2; no longer R10.1, R11.1, R37.2, R38.2, R39.2
Other:
- moved on the sheet: C10, C11, C6, C7, C8, C9

Commit message: routing
Parts:
- removed QA4: MMPQ2222A, nest_interface:MMPQ2222A
- added Q1, Q2: (no value), nest_interface:TRANSISTOR_NPNSOT23
Connections:
- removed net N$35: R33.1
- removed net N$36: R35.1
- removed net N$59: QA1.B3, RA4.22
- removed net N$61: QA2.B1, RA4.20
- removed net N$62: QA2.B2, RA4.19
- removed net N$63: QA2.B3, RA4.18
- removed net N$64: QA2.B4, RA4.17
- removed net N$66: QA3.B2, RA4.15
- removed net N$67: QA3.B3, RA4.14
- removed net N$68: QA3.B4, RA4.13
- new net N$16: QA1.B3, RA4.23
- new net N$17: QA2.B2, RA4.18
- new net N$25: QA2.B3, RA4.19
- new net N$26: QA2.B4, RA4.20
- new net N$28: QA3.B1, RA4.13
- new net N$29: QA3.B2, RA4.14
- new net N$30: QA3.B3, RA4.15
- new net N$31: Q1.B, R33.1
- new net N$32: Q2.B, R35.1
- new net N$5: QA2.B1, RA4.17
- net GND: now also Q1.E, Q2.E; no longer QA4.E1, QA4.E2
- net N$37: now also QA1.B4; no longer QA1.B1
- net N$58: now also RA4.22; no longer RA4.23
- net N$60: now also QA1.B1; no longer QA1.B4
- net N$65: now also QA3.B4; no longer QA3.B1
- net TSTAT1_DOWN_IN: now also RA6.3; no longer RA6.6
- net TSTAT1_DOWN_OUT: now also QA2.C3; no longer QA2.C2
- net TSTAT1_ENTER_IN: now also RA6.2; no longer RA6.7
- net TSTAT1_ENTER_OUT: now also QA2.C2; no longer QA2.C3
- net TSTAT1_ESC_IN: now also RA6.5; no longer RA6.4
- net TSTAT1_ESC_OUT: now also QA1.C1; no longer QA1.C4
- net TSTAT1_HELP_IN: now also RA6.4; no longer RA6.5
- net TSTAT1_HELP_OUT: now also QA2.C4; no longer QA2.C1
- net TSTAT1_MENU_IN: now also RA6.7; no longer RA6.2
- net TSTAT1_MENU_OUT: now also QA1.C3; no longer QA1.C2
- net TSTAT1_ON/OFF_IN: now also RA6.8; no longer RA6.1
- net TSTAT1_ON/OFF_OUT: now also QA1.C4; no longer QA1.C1
- net TSTAT1_UP_IN: now also RA6.6; no longer RA6.3
- net TSTAT1_UP_OUT: now also QA1.C2; no longer QA1.C3
- net TSTAT2_DOWN_IN: now also RA6.14; no longer RA6.13
- net TSTAT2_DOWN_OUT: now also Q1.C; no longer QA4.C1
- net TSTAT2_ENTER_IN: now also RA6.15; no longer RA6.14
- net TSTAT2_ENTER_OUT: now also Q2.C; no longer QA4.C2
- net TSTAT2_ESC_IN: now also RA6.12; no longer RA6.11
- net TSTAT2_ESC_OUT: now also QA3.C2; no longer QA3.C3
- net TSTAT2_ESC_OUT_PIN: now also RA5.11; no longer RA5.10
- net TSTAT2_HELP_IN: now also RA6.13; no longer RA6.12
- net TSTAT2_HELP_OUT: now also QA3.C1; no longer QA3.C4
- net TSTAT2_HELP_OUT_PIN: now also RA5.12; no longer RA5.9
- net TSTAT2_MENU_IN: now also RA6.10; no longer RA6.9
- net TSTAT2_MENU_OUT: now also QA3.C4; no longer QA3.C1
- net TSTAT2_MENU_OUT_PIN: now also RA5.9; no longer RA5.12
- net TSTAT2_ON/OFF_IN: now also RA6.9; no longer RA6.8
- net TSTAT2_ON/OFF_OUT: now also QA2.C1; no longer QA2.C4
- net TSTAT2_UP_IN: now also RA6.11; no longer RA6.10
- net TSTAT2_UP_OUT: now also QA3.C3; no longer QA3.C2
- net TSTAT2_UP_OUT_PIN: now also RA5.10; no longer RA5.11

Commit message: cleaned up the nib schematic
Parts:
- removed J23, J24: CONN_BLOCK_8, nest_interface:CONN_BLOCK_8
- removed J25: MOLEX_MICRO_USB_B_047346, nest_interface:MOLEX_MICRO_USB_B_047346
- removed J30: PINH2X12, SparkFun:PINH2X12
- removed JP1: (no value), pinhead:PINHD-2X10
- removed RA6: 766161104GP, nest_interface:766161104GP
- removed U20: MSP430F1611IPM, hijack:MSP430F1611IPM
- added J10, J9: CONN_BLOCK_2, nest_interface:CONN_BLOCK_2
- added J16: CONN_BLOCK_7, nest_interface:CONN_BLOCK_7
- added J18, J19, J20, J21: CONN_BLOCK_8, nest_interface:CONN_BLOCK_8
- added QA5: ALD1107, nest_interface:ALD1107
- added RA3: VSSR2403103, nest_interface:VSSR2403103
- J14, J15: value CONN_BLOCK_2 -> CONN_BLOCK_3; device nest_interface:CONN_BLOCK_2 -> nest_interface:CONN_BLOCK_3
- J17: value CONN_BLOCK_3 -> CONN_BLOCK_7; device nest_interface:CONN_BLOCK_3 -> nest_interface:CONN_BLOCK_7
- J2: value CONN_BLOCK_2 -> MOLEX_MICRO_USB_B_047346; device nest_interface:CONN_BLOCK_2 -> nest_interface:MOLEX_MICRO_USB_B_047346
- J3: value CONN_BLOCK_3 -> (none); device nest_interface:CONN_BLOCK_3 -> pinhead:PINHD-2X10
- J4: value PJ-036A-SMT -> PINH2X12; device nest_interface:PJ-036A-SMT -> SparkFun:PINH2X12
- J5: value CONN_BLOCK_8 -> PJ-036A-SMT; device nest_interface:CONN_BLOCK_8 -> nest_interface:PJ-036A-SMT
- J6: value CONN_BLOCK_8 -> CONN_BLOCK_2; device nest_interface:CONN_BLOCK_8 -> nest_interface:CONN_BLOCK_2
- J7, J8: value CONN_BLOCK_7 -> CONN_BLOCK_2; device nest_interface:CONN_BLOCK_7 -> nest_interface:CONN_BLOCK_2
- RA4: value VSSR2403103 -> 766161104GP; device nest_interface:VSSR2403103 -> nest_interface:766161104GP
- S2: value EVQP2 -> (none); device berkeley-epic:EVQP2 -> SparkFun:SWITCH-SPSTPTH
- S4: value (none) -> EVQP2; device SparkFun:SWITCH-SPSTPTH -> berkeley-epic:EVQP2
- U1: value FT232RL -> EPIC-CORE_A; device ftdichip:FT232RL -> berkeley-epic:EPIC-CORE_A
- U2: value EPIC-CORE_A -> MSP430F1611IPM; device berkeley-epic:EPIC-CORE_A -> hijack:MSP430F1611IPM
- U3: value MPC1825 -> FT232RL; device nest_interface:MPC1825 -> ftdichip:FT232RL
- U4: value PCA9575 -> FT232RL; device nest_interface:PCA9575 -> ftdichip:FT232RL
- U5: value PCA9575 -> MPC1825; device nest_interface:PCA9575 -> nest_interface:MPC1825
- U6: value FT232RL -> TC1262; device ftdichip:FT232RL -> nest_interface:TC1262
- U7: value TC1262 -> PCA9575; device nest_interface:TC1262 -> nest_interface:PCA9575
- U8: value ALD1107 -> PCA9575; device nest_interface:ALD1107 -> nest_interface:PCA9575
- renumbered U10 to QA7, U11 to QA8, U9 to QA6
Connections:
- new net TSTAT1_SPEAKER_IN: J12.2
- new net TSTAT1_SPEAKER_OUT: J12.1
- new net TSTAT2_SPEAKER_IN: J13.2
- new net TSTAT2_SPEAKER_OUT: J13.1
- net #KEYPAD_ENABLE: now also QA5.G1, QA5.G2, QA5.G3, QA5.G4, U1.P5.2; no longer U2.P5.2, U8.G1, U8.G2, U8.G3, U8.G4
- net 5.6V_SUPPLY: now also J7.2, U5.VIN, U6.VIN; no longer J11.2, U3.VIN, U7.VIN
- net 5V: now also J8.2, J9.2, U6.VOUT; no longer J12.2, J13.2, U7.VOUT
- net COMMON: now also J5.COMMON, J6.2; no longer J2.2, J4.COMMON
- net COOLING1_PIN: now also U1.P1.6; no longer U2.P1.6
- net COOLING2_PIN: now also U1.P2.3; no longer U2.P2.3
- net EPIC_ADC1: now also J3.18, U1.ADC1; no longer JP1.18, U2.ADC1
- net EPIC_ADC2: now also J3.16, U1.ADC2; no longer JP1.16, U2.ADC2
- net EPIC_ADC3: now also J3.14, U1.ADC3; no longer JP1.14, U2.ADC3
- net EPIC_ADC4: now also J3.12, U1.ADC4; no longer JP1.12, U2.ADC4
- net EPIC_ADC5: now also J3.10, U1.ADC5; no longer JP1.10, U2.ADC5
- net EPIC_ADC6/DAC0: now also J3.8, U1.ADC6/DAC0; no longer JP1.8, U2.ADC6/DAC0
- net EPIC_ADC7/DAC1: now also J3.6, U1.ADC7/DAC1; no longer JP1.6, U2.ADC7/DAC1
- net EPIC_MISO0: now also J3.13, U1.MISO0; no longer JP1.13, U2.MISO0
- net EPIC_P2.0: now also J3.1, U1.P2.0; no longer JP1.1, U2.P2.0
- net EPIC_P2.4: now also J3.5, U1.ONEWIRE; no longer JP1.5, U2.ONEWIRE
- net EPIC_P2.7: now also J3.3, U1.I2C0/~SPI0; no longer JP1.3, U2.I2C0/~SPI0
- net EPIC_P5.7: now also J3.7, U1.P5.7; no longer JP1.7, U2.P5.7
- net EPIC_STE0: now also J3.9, U1.STE0; no longer JP1.9, U2.STE0
- net EPIC_UART0RX: now also J3.19, U1.UART0RX; no longer JP1.19, U2.UART0RX
- net EPIC_UART0TX: now also J3.17, U1.UART0TX; no longer JP1.17, U2.UART0TX
- net FAN_PIN: now also U1.P1.5; no longer U2.P1.5
- net G: now also J14.1; no longer J3.1
- net GND: now also J10.1, J18.1, J19.1, J2.GND, J20.1, J21.1, J3.20, J7.1, J8.1, J9.1, QA5.GND, RA4.OUT, S4.P$1, S4.P$3, U1.AGND, U1.GND1, U1.GND2, U1.GND3, U2.AVSS, U2.DVSS1, U2.VEREF+, U2.VREF-/VEREF-, U2.XT2IN, U3.GND@1, U3.GND@2, U3.GND@A, U3.TEST, U4.GND@1, U4.GND@2, U4.GND@A, U4.TEST, U7.ADDR3, U7.P0_7, U7.P1_7, U8.ADDR2, U8.ADDR3; no longer J12.1, J13.1, J14.1, J15.1, J23.1, J24.1, J25.GND, J5.1, J6.1, JP1.20, RA5.OUT, S2.P$1, S2.P$3, U1.GND, U1.GND@1, U1.GND@2, U1.GND@A, U1.TEST, U2.AGND, U2.GND1, U2.GND2, U2.GND3, U20.AVSS, U20.DVSS1, U20.VEREF+, U20.VREF-/VEREF-, U20.XT2IN, U4.ADDR3, U4.P0_7, U4.P1_7, U5.ADDR2, U5.ADDR3, U6.GND@1, U6.GND@2, U6.GND@A, U6.TEST
- net HEATING1_PIN: now also U1.P1.7; no longer U2.P1.7
- net HEATING2_PIN: now also U1.P2.6; no longer U2.P2.6
- net I2C_SCL: now also J3.15, U1.SCLK0/SCL, U2.P3.3/UCLK0/SCL, U7.SCL, U8.SCL; no longer JP1.15, U2.SCLK0/SCL, U20.P3.3/UCLK0/SCL, U4.SCL, U5.SCL
- net I2C_SDA: now also J3.11, U1.MOSI0/SDA, U2.P3.1/MOSI0/SDA, U7.SDA, U8.SDA; no longer JP1.11, U2.MOSI0/SDA, U20.P3.1/MOSI0/SDA, U4.SDA, U5.SDA
- net LCDP_MISO0: now also J4.16, U2.P3.2/MISO0; no longer J30.16, U20.P3.2/MISO0
- net LCDP_P2.4: now also J4.4, U2.P2.4/CA1/TA2; no longer J30.4, U20.P2.4/CA1/TA2
- net LCDP_P2.7: now also U2.P2.7/TA0; no longer U20.P2.7/TA0
- net LCDP_STE0: now also J4.18, U2.P3.0/STE0; no longer J30.18, U20.P3.0/STE0
- net LCDP_URXD0: now also J4.12, U2.P3.5/URXD0; no longer J30.12, U20.P3.5/URXD0
- net LCDP_UTXD0: now also J4.14, U2.P3.4/UTXD0; no longer J30.14, U20.P3.4/UTXD0
- net N$10: now also U3.CBUS0; no longer U1.CBUS0
- net N$11: now also U3.CBUS1; no longer U1.CBUS1
- net N$12: now also U1.UART1TX, U3.RXD; no longer U1.RXD, U2.UART1TX
- net N$14: now also U1.TCK, U3.!DTR; no longer U1.!DTR, U2.TCK
- net N$15: now also U3.3V3OUT, U3.VCCIO; no longer U1.3V3OUT, U1.VCCIO
- net N$16: now also RA3.23; no longer RA4.23
- net N$17: now also RA3.18; no longer RA4.18
- net N$18: now also U1.AVDD; no longer U2.AVDD
- net N$22: now also U1.LED3; no longer U2.LED3
- net N$23: now also U1.LED2; no longer U2.LED2
- net N$24: now also U1.LED1; no longer U2.LED1
- net N$25: now also RA3.19; no longer RA4.19
- net N$26: now also RA3.20; no longer RA4.20
- net N$28: now also RA3.13; no longer RA4.13
- net N$29: now also RA3.14; no longer RA4.14
- net N$3: now also U3.USBDM; no longer U1.USBDM
- net N$30: now also RA3.15; no longer RA4.15
- net N$37: now also RA3.24; no longer RA4.24
- net N$38: now also U2.XIN; no longer U20.XIN
- net N$39: now also J2.VCC; no longer J25.VCC
- net N$4: now also U3.USBDP; no longer U1.USBDP
- net N$40: now also J2.D-, U4.USBDM; no longer J25.D-, U6.USBDM
- net N$41: now also J2.D+, U4.USBDP; no longer J25.D+, U6.USBDP
- net N$43: now also U4.VCC; no longer U6.VCC
- net N$44: now also U4.CBUS0; no longer U6.CBUS0
- net N$45: now also U4.CBUS1; no longer U6.CBUS1
- net N$48: now also U2.P3.7/URXD1, U4.TXD; no longer U20.P3.6/UTXD1, U6.TXD
- net N$49: now also U2.P3.6/UTXD1, U4.RXD; no longer U20.P3.7/URXD1, U6.RXD
- net N$5: now also RA3.17; no longer RA4.17
- net N$50: now also U2.TCK, U4.!DTR; no longer U20.TCK, U6.!DTR
- net N$51: now also U4.3V3OUT, U4.VCCIO; no longer U6.3V3OUT, U6.VCCIO
- net N$52: now also U2.XOUT; no longer U20.XOUT
- net N$54: now also U2.P2.5/ROSC; no longer U20.P2.5/ROSC
- net N$56: now also U2.P2.1/TAINCLK; no longer U20.P2.1/TAINCLK
- net N$57: now also U2.P2.2/CAOUT/TA0/BSLRX; no longer U20.P2.2/CAOUT/TA0/BSLRX
- net N$58: now also RA3.22; no longer RA4.22
- net N$6: now also U3.VCC; no longer U1.VCC
- net N$60: now also RA3.21; no longer RA4.21
- net N$65: now also RA3.16; no longer RA4.16
- net N$8: now also U2.P2.0/ACLK; no longer U20.P2.0/ACLK
- net N$9: now also U1.UART1RX, U3.TXD; no longer U1.TXD, U2.UART1RX
- net P1.6: now also J4.10, U2.P1.6/TA1; no longer J30.10, U20.P1.6/TA1
- net P1.7: now also J4.8, U2.P1.7/TA2; no longer J30.8, U20.P1.7/TA2
- net P2.3: now also J4.6, U2.P2.3/CA0/TA1; no longer J30.6, U20.P2.3/CA0/TA1
- net P2.6: now also J4.2, U2.P2.6/ADC12CLK/DMAE0; no longer J30.2, U20.P2.6/ADC12CLK/DMAE0
- net P5.0: now also J4.1, U2.P5.0/STE1; no longer J30.1, U20.P5.0/STE1
- net P5.1: now also J4.3, U2.P5.1/MOSI1; no longer J30.3, U20.P5.1/MOSI1
- net P5.2: now also J4.5, U2.P5.2/MISO1; no longer J30.5, U20.P5.2/MISO1
- net P5.3: now also J4.7, U2.P5.3/UCLK1; no longer J30.7, U20.P5.3/UCLK1
- net P5.4: now also J4.9, U2.P5.4/MCLK; no longer J30.9, U20.P5.4/MCLK
- net P5.5: now also U2.P5.5/SMCLK; no longer U20.P5.5/SMCLK
- net P5.6: now also J4.11, U2.P5.6/ACLK; no longer J30.11, U20.P5.6/ACLK
- net P5.7: now also J4.13, U2.P5.7/TBOUTH/SVSOUT; no longer J30.13, U20.P5.7/TBOUTH/SVSOUT
- net P6.0: now also J4.15, U2.P6.0/A0; no longer J30.15, U20.P6.0/A0
- net P6.1: now also J4.17, U2.P6.1/A1; no longer J30.17, U20.P6.1/A1
- net P6.2: now also J4.19, U2.P6.2/A2; no longer J30.19, U20.P6.2/A2
- net P6.3: now also J4.21, U2.P6.3/A3; no longer J30.21, U20.P6.3/A3
- net P6.4: now also J4.23, U2.P6.4/A4; no longer J30.23, U20.P6.4/A4
- net P6.5: now also J4.24, U2.P6.5/A5; no longer J30.24, U20.P6.5/A5
- net P6.6: now also J4.22, U2.P6.6/A6/DAC0; no longer J30.22, U20.P6.6/A6/DAC0
- net P6.7: now also J4.20, U2.P6.7/A7/DAC1/SVSIN; no longer J30.20, U20.P6.7/A7/DAC1/SVSIN
- net RADIO_SFD: now also J3.4, U1.RADIO_SFD; no longer JP1.4, U2.RADIO_SFD
- net RH: now also J5.24V, J6.1; no longer J2.1, J4.24V
- net RST: now also S3.P$2, S3.P$4, U1.RST/NMI; no longer S2.P$2, S2.P$4, U2.RST/NMI
- net RST1: now also S2.O, S4.P$2, S4.P$4, U2.RST/NMI; no longer S3.P$2, S3.P$4, S4.O, U20.RST/NMI
- net RST_USB: now also U3.!RTS; no longer U1.!RTS
- net RST_USB1: now also S2.P, U4.!RTS; no longer S4.P, U6.!RTS
- net STAR: now also J15.1; no longer J17.1
- net STAR_PIN: now also U1.P2.1; no longer U2.P2.1
- net TSTAT1_DOWN_IN: now also J18.3, RA5.3, U7.P0_1; no longer J5.3, RA6.3, U4.P0_1
- net TSTAT1_DOWN_OUT: now also J20.3; no longer J23.3
- net TSTAT1_DOWN_OUT_PIN: now also RA3.6, RA4.3, U8.P0_5; no longer RA4.6, RA5.3, U5.P0_5
- net TSTAT1_ENTER_IN: now also J18.2, RA5.2, U7.P0_0; no longer J5.2, RA6.2, U4.P0_0
- net TSTAT1_ENTER_OUT: now also J20.2; no longer J23.2
- net TSTAT1_ENTER_OUT_PIN: now also RA3.7, RA4.2, U8.P0_6; no longer RA4.7, RA5.2, U5.P0_6
- net TSTAT1_ESC_IN: now also J18.5, QA5.S4, RA5.5, U7.P0_3; no longer J5.5, RA6.5, U4.P0_3, U8.S4
- net TSTAT1_ESC_OUT: now also J20.5, QA5.D4; no longer J23.5, U8.D4
- net TSTAT1_ESC_OUT_PIN: now also RA3.4, RA4.5, U8.P0_3; no longer RA4.4, RA5.5, U5.P0_3
- net TSTAT1_HELP_IN: now also J18.4, RA5.4, U7.P0_2; no longer J5.4, RA6.4, U4.P0_2
- net TSTAT1_HELP_OUT: now also J20.4; no longer J23.4
- net TSTAT1_HELP_OUT_PIN: now also RA3.5, RA4.4, U8.P0_4; no longer RA4.5, RA5.4, U5.P0_4
- net TSTAT1_LCD_DB4: now also J16.4; no longer J7.4
- net TSTAT1_LCD_DB4_PIN: now also U2.P4.0/TB0; no longer U20.P4.0/TB0
- net TSTAT1_LCD_DB5: now also J16.5; no longer J7.5
- net TSTAT1_LCD_DB5_PIN: now also U2.P4.1/TB1; no longer U20.P4.1/TB1
- net TSTAT1_LCD_DB6: now also J16.6; no longer J7.6
- net TSTAT1_LCD_DB6_PIN: now also U2.P4.2/TB2; no longer U20.P4.2/TB2
- net TSTAT1_LCD_DB7: now also J16.7; no longer J7.7
- net TSTAT1_LCD_DB7_PIN: now also U2.P4.3/TB3; no longer U20.P4.3/TB3
- net TSTAT1_LCD_E: now also J16.3; no longer J7.3
- net TSTAT1_LCD_E_PIN: now also U2.P1.3/TA2; no longer U20.P1.3/TA2
- net TSTAT1_LCD_R/W: now also J16.2; no longer J7.2
- net TSTAT1_LCD_R/W_PIN: now also U2.P1.4/SMCLK; no longer U20.P1.4/SMCLK
- net TSTAT1_LCD_RS: now also J16.1; no longer J7.1
- net TSTAT1_LCD_RS_PIN: now also U2.P1.5/TA0; no longer U20.P1.5/TA0
- net TSTAT1_MENU_IN: now also J18.7, QA5.S2, RA5.7, U7.P0_5; no longer J5.7, RA6.7, U4.P0_5, U8.S2
- net TSTAT1_MENU_OUT: now also J20.7, QA5.D2; no longer J23.7, U8.D2
- net TSTAT1_MENU_OUT_PIN: now also RA3.2, RA4.7, U8.P0_1; no longer RA4.2, RA5.7, U5.P0_1
- net TSTAT1_ON/OFF_IN: now also J18.8, QA5.S1, RA5.8, U7.P0_6; no longer J5.8, RA6.8, U4.P0_6, U8.S1
- net TSTAT1_ON/OFF_OUT: now also J20.8, QA5.D1; no longer J23.8, U8.D1
- net TSTAT1_ON/OFF_OUT_PIN: now also RA3.1, RA4.8, U8.P0_0; no longer RA4.1, RA5.8, U5.P0_0
- net TSTAT1_UP_IN: now also J18.6, QA5.S3, RA5.6, U7.P0_4; no longer J5.6, RA6.6, U4.P0_4, U8.S3
- net TSTAT1_UP_OUT: now also J20.6, QA5.D3; no longer J23.6, U8.D3
- net TSTAT1_UP_OUT_PIN: now also RA3.3, RA4.6, U8.P0_2; no longer RA4.3, RA5.6, U5.P0_2
- net TSTAT2_DOWN_IN: now also J19.3, RA5.14, U7.P1_5; no longer J6.3, RA6.14, U4.P1_5
- net TSTAT2_DOWN_OUT: now also J21.3; no longer J24.3
- net TSTAT2_DOWN_OUT_PIN: now also RA4.13, U8.P1_5; no longer RA5.13, U5.P1_5
- net TSTAT2_ENTER_IN: now also J19.2, RA5.15, U7.P1_6; no longer J6.2, RA6.15, U4.P1_6
- net TSTAT2_ENTER_OUT: now also J21.2; no longer J24.2
- net TSTAT2_ENTER_OUT_PIN: now also RA4.14, U8.P1_6; no longer RA5.14, U5.P1_6
- net TSTAT2_ESC_IN: now also J19.5, RA5.12, U7.P1_3; no longer J6.5, RA6.12, U4.P1_3
- net TSTAT2_ESC_OUT: now also J21.5; no longer J24.5
- net TSTAT2_ESC_OUT_PIN: now also RA3.11, U8.P1_3; no longer RA5.11, U5.P1_3
- net TSTAT2_HELP_IN: now also J19.4, RA5.13, U7.P1_4; no longer J6.4, RA6.13, U4.P1_4
- net TSTAT2_HELP_OUT: now also J21.4; no longer J24.4
- net TSTAT2_HELP_OUT_PIN: now also RA3.12, U8.P1_4; no longer RA5.12, U5.P1_4
- net TSTAT2_LCD_DB4: now also J17.4; no longer J8.4
- net TSTAT2_LCD_DB4_PIN: now also U2.P4.4/TB4; no longer U20.P4.4/TB4
- net TSTAT2_LCD_DB5: now also J17.5; no longer J8.5
- net TSTAT2_LCD_DB5_PIN: now also U2.P4.5/TB5; no longer U20.P4.5/TB5
- net TSTAT2_LCD_DB6: now also J17.6; no longer J8.6
- net TSTAT2_LCD_DB6_PIN: now also U2.P4.6/TB6; no longer U20.P4.6/TB6
- net TSTAT2_LCD_DB7: now also J17.7; no longer J8.7
- net TSTAT2_LCD_DB7_PIN: now also U2.P4.7/TBCLK; no longer U20.P4.7/TBCLK
- net TSTAT2_LCD_E: now also J17.3; no longer J8.3
- net TSTAT2_LCD_E_PIN: now also U2.P1.2/TA1; no longer U20.P1.2/TA1
- net TSTAT2_LCD_R/W: now also J17.2; no longer J8.2
- net TSTAT2_LCD_R/W_PIN: now also U2.P1.1/TA0/BSLTX; no longer U20.P1.1/TA0/BSLTX
- net TSTAT2_LCD_RS: now also J17.1; no longer J8.1
- net TSTAT2_LCD_RS_PIN: now also U2.P1.0/TACLK; no longer U20.P1.0/TACLK
- net TSTAT2_MENU_IN: now also J19.7, RA5.10, U7.P1_1; no longer J6.7, RA6.10, U4.P1_1
- net TSTAT2_MENU_OUT: now also J21.7; no longer J24.7
- net TSTAT2_MENU_OUT_PIN: now also RA3.9, U8.P1_1; no longer RA5.9, U5.P1_1
- net TSTAT2_ON/OFF_IN: now also J19.8, RA5.9, U7.P1_0; no longer J6.8, RA6.9, U4.P1_0
- net TSTAT2_ON/OFF_OUT: now also J21.8; no longer J24.8
- net TSTAT2_ON/OFF_OUT_PIN: now also RA3.8, RA4.1, U8.P1_0; no longer RA4.8, RA5.1, U5.P1_0
- net TSTAT2_UP_IN: now also J19.6, RA5.11, U7.P1_2; no longer J6.6, RA6.11, U4.P1_2
- net TSTAT2_UP_OUT: now also J21.6; no longer J24.6
- net TSTAT2_UP_OUT_PIN: now also RA3.10, U8.P1_2; no longer RA5.10, U5.P1_2
- net TSTAT_IN_I2C_INT: now also U1.P1.2, U7.#INT; no longer U2.P1.2, U4.#INT
- net TSTAT_IN_I2C_RST: now also U1.P5.0, U7.#RESET; no longer U2.P5.0, U4.#RESET
- net TSTAT_OUT_I2C_RST: now also U1.P5.1, U8.#RESET; no longer U2.P5.1, U5.#RESET
- net VCC: now also J10.2, J11.2, J3.2, QA5.VCC, RA5.OUT, U1.DVDD, U1.FLASH_WP, U1.FVDD, U1.RVDD, U2.AVCC, U2.DVCC, U5.VOUT, U7.ADDR0, U7.ADDR1, U7.ADDR2, U7.P0_VCC, U7.P1_VCC, U7.VCC, U8.ADDR0, U8.ADDR1, U8.P0_VCC, U8.P1_VCC; no longer J14.2, J15.2, JP1.2, RA6.OUT, U2.DVDD, U2.FLASH_WP, U2.FVDD, U2.RVDD, U20.AVCC, U20.DVCC, U3.VOUT, U4.ADDR0, U4.ADDR1, U4.ADDR2, U4.P0_VCC, U4.P1_VCC, U4.VCC, U5.ADDR0, U5.ADDR1, U5.P0_VCC, U5.P1_VCC, U5.VCC
- net W1: now also J14.3; no longer J3.3
- net W2: now also J15.3; no longer J17.3
- net Y1: now also J14.2; no longer J3.2
- net Y2: now also J15.2; no longer J17.2

Commit message: updated bom
Changed lines of the file:
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@@
 </classes>
 <parts>
-<part name="FRAME2" library="frames" deviceset="LETTER_L" device=""/>
 <part name="U3" library="ftdichip" deviceset="FT232R" device="L"/>
 <part name="J1" library="nest_interface" deviceset="MOLEX_MICRO_USB_B_047346" device=""/>
@@
 <part name="GND24" library="supply1" deviceset="GND" device=""/>
 <part name="GND25" library="supply1" deviceset="GND" device=""/>
-<part name="FRAME3" library="frames" deviceset="LETTER_L" device=""/>
 <part name="R33" library="rcl" deviceset="R-US_" device="R0603" value="10k"/>
 <part name="GND31" library="supply1" deviceset="GND" device=""/>
@@
 <part name="GND40" library="supply1" deviceset="GND" device=""/>
 <part name="P+8" library="SparkFun" deviceset="VCC" device=""/>
-<part name="FRAME4" library="frames" deviceset="LETTER_L" device=""/>
 <part name="RE4" library="nest_interface" deviceset="RT314524" device=""/>
 <part name="RE5" library="nest_interface" deviceset="RT314524" device=""/>
@@
 <part name="J15" library="nest_interface" deviceset="CONN_BLOCK_3" device=""/>
 <part name="S1" library="SparkFun" deviceset="SWITCH-SPST" device="PTH"/>
-<part name="FRAME5" library="frames" deviceset="LETTER_L" device=""/>
 <part name="QA5" library="nest_interface" deviceset="ALD1107" device=""/>
 <part name="P+20" library="SparkFun" deviceset="VCC" device=""/>
@@
 <part name="P+35" library="SparkFun" deviceset="VCC" device=""/>
 <part name="GND66" library="supply1" deviceset="GND" device=""/>
-<part name="FRAME6" library="frames" deviceset="LETTER_L" device=""/>
 <part name="U7" library="nest_interface" deviceset="PCA9575" device=""/>
 <part name="U8" library="nest_interface" deviceset="PCA9575" device=""/>
@@
 <part name="GND69" library="supply1" deviceset="GND" device=""/>
 <part name="R72" library="rcl" deviceset="R-US_" device="R0603" value="100k"/>
-<part name="FRAME7" library="frames" deviceset="LETTER_L" device=""/>
 <part name="U2" library="hijack" deviceset="MSP430F1611" device="IPM"/>
 <part name="P+42" library="SparkFun" deviceset="VCC" device=""/>
@@
 <part name="C17" library="rcl" deviceset="C-EU" device="C0603" value="0.1u"/>
 <part name="GND81" library="supply1" deviceset="GND" device=""/>
-<part name="FRAME8" library="frames" deviceset="LETTER_L" device=""/>
 <part name="RA1" library="nest_interface" deviceset="VSSR2403103" device=""/>
 <part name="GND87" library="supply1" deviceset="GND" device=""/>
@@
 <part name="J13" library="nest_interface" deviceset="CONN_BLOCK_2" device=""/>
 <part name="FRAME1" library="nest_interface" deviceset="LETTER_L" device=""/>
+<part name="FRAME2" library="nest_interface" deviceset="LETTER_L" device=""/>
+<part name="FRAME3" library="nest_interface" deviceset="LETTER_L" device=""/>
+<part name="FRAME4" library="nest_interface" deviceset="LETTER_L" device=""/>
+<part name="FRAME5" library="nest_interface" deviceset="LETTER_L" device=""/>
+<part name="FRAME6" library="nest_interface" deviceset="LETTER_L" device=""/>
+<part name="FRAME7" library="nest_interface" deviceset="LETTER_L" device=""/>
+<part name="FRAME8" library="nest_interface" deviceset="LETTER_L" device=""/>
 </parts>
 <sheets>
@@
 </plain>
 <instances>
-<instance part="FRAME4" gate="G$1" x="0" y="0"/>
-<instance part="FRAME4" gate="G$2" x="147.32" y="0"/>
 <instance part="RE1" gate="G$1" x="40.64" y="157.48"/>
 <instance part="RE2" gate="G$1" x="40.64" y="111.76"/>
@@
 <instance part="GND45" gate="1" x="172.72" y="96.52"/>
 <instance part="GND46" gate="1" x="172.72" y="50.8"/>
+<instance part="FRAME2" gate="G$1" x="0" y="0"/>
+<instance part="FRAME2" gate="G$2" x="147.32" y="0"/>
 </instances>
 <busses>
@@
 </plain>
 <instances>
-<instance part="FRAME3" gate="G$1" x="0" y="0"/>
-<instance part="FRAME3" gate="G$2" x="147.32" y="0"/>
 <instance part="R33" gate="G$1" x="43.18" y="30.48" rot="R180"/>
 <instance part="GND31" gate="1" x="99.06" y="17.78"/>
@@
 <instance part="Q1" gate="G$1" x="53.34" y="30.48"/>
 <instance part="Q2" gate="G$1" x="119.38" y="30.48"/>
+<instance part="FRAME3" gate="G$1" x="0" y="0"/>
+<instance part="FRAME3" gate="G$2" x="147.32" y="0"/>
 </instances>
 <busses>
@@
 </plain>
 <instances>
-<instance part="FRAME5" gate="G$1" x="0" y="0"/>
-<instance part="FRAME5" gate="G$2" x="147.32" y="0"/>
 <instance part="QA5" gate="G$1" x="73.66" y="147.32"/>
 <instance part="P+20" gate="1" x="114.3" y="152.4"/>
@@
 <instance part="RA5" gate="G$1" x="198.12" y="114.3"/>
 <instance part="P+45" gate="1" x="205.74" y="116.84"/>
+<instance part="FRAME4" gate="G$1" x="0" y="0"/>
+<instance part="FRAME4" gate="G$2" x="147.32" y="0"/>
 </instances>
 <busses>
@@
 </plain>
 <instances>
-<instance part="FRAME2" gate="G$1" x="0" y="0"/>
-<instance part="FRAME2" gate="G$2" x="147.32" y="0"/>
 <instance part="U3" gate="1" x="88.9" y="53.34"/>
 <instance part="J1" gate="G$1" x="17.78" y="40.64"/>
@@
 <instance part="GND40" gate="1" x="60.96" y="134.62"/>
 <instance part="P+8" gate="1" x="60.96" y="165.1"/>
+<instance part="FRAME5" gate="G$1" x="0" y="0"/>
+<instance part="FRAME5" gate="G$2" x="147.32" y="0"/>
 </instances>
 <busses>
@@
 </plain>
 <instances>
-<instance part="FRAME6" gate="G$1" x="0" y="0"/>
-<instance part="FRAME6" gate="G$2" x="147.32" y="0"/>
 <instance part="U7" gate="G$1" x="71.12" y="104.14"/>
 <instance part="U8" gate="G$1" x="185.42" y="104.14"/>
@@
 <instance part="R101" gate="G$1" x="76.2" y="22.86" rot="R270"/>
 <instance part="R102" gate="G$1" x="86.36" y="22.86" rot="R270"/>
+<instance part="FRAME6" gate="G$1" x="0" y="0"/>
+<instance part="FRAME6" gate="G$2" x="147.32" y="0"/>
 </instances>
 <busses>
@@
 </plain>
 <instances>
-<instance part="FRAME7" gate="G$1" x="0" y="0"/>
-<instance part="FRAME7" gate="G$2" x="147.32" y="0"/>
 <instance part="U2" gate="G$1" x="182.88" y="116.84"/>
 <instance part="P+42" gate="1" x="180.34" y="177.8"/>
@@
 <instance part="P+48" gate="1" x="86.36" y="154.94"/>
 <instance part="J4" gate="G$1" x="38.1" y="137.16"/>
+<instance part="FRAME7" gate="G$1" x="0" y="0"/>
+<instance part="FRAME7" gate="G$2" x="147.32" y="0"/>
 </instances>
 <busses>
@@
 </plain>
 <instances>
-<instance part="FRAME8" gate="G$1" x="0" y="0"/>
-<instance part="FRAME8" gate="G$2" x="147.32" y="0"/>
 <instance part="RA1" gate="G$1" x="96.52" y="121.92"/>
 <instance part="GND87" gate="1" x="83.82" y="104.14"/>
@@
 <instance part="RA7" gate="G$1" x="195.58" y="99.06"/>
 <instance part="GND16" gate="1" x="182.88" y="83.82"/>
+<instance part="FRAME8" gate="G$1" x="0" y="0"/>
+<instance part="FRAME8" gate="G$2" x="147.32" y="0"/>
 </instances>
 <busses>

Commit message: more schematic updates
Parts:
- L2: DIGIKEY (none) -> 240-2373-1-ND
- Q1, Q2: DIGIKEY (none) -> 568-1636-1-ND
- S1, S2: DIGIKEY (none) -> EG1903-ND
- U3, U4: DIGIKEY (none) -> 768-1007-1-ND
- renumbered R10 to R2122, R101 to R1322, R102 to R1422, R11 to R2322, R33 to R1522, R35 to R1622, R6 to R1722, R66 to R2622, R67 to R2722, R7 to R1822, R72 to R2522, R73 to R622, R74 to R722, R75 to R1222, R76 to R1122, R77 to R2822, R78 to R1022, R79 to R922, R8 to R1922, R80 to R822, R9 to R2022, R99 to R2422
Connections:
- net #KEYPAD_ENABLE: now also QA8.G3, QA8.G4
- net TSTAT1_SPEAKER_IN: now also QA8.S4
- net TSTAT1_SPEAKER_OUT: now also QA8.D4
- net TSTAT2_SPEAKER_IN: now also QA8.S3
- net TSTAT2_SPEAKER_OUT: now also QA8.D3

Commit message: no airwires!!!!!
Parts:
- J4: value PINH2X12 -> (none); device SparkFun:PINH2X12 -> pinhead:PINHD-2X10
Connections:
- net LCDP_MISO0: no longer J4.16
- net LCDP_P2.4: no longer J4.4
- net LCDP_STE0: no longer J4.18
- net LCDP_URXD0: no longer J4.12
- net LCDP_UTXD0: no longer J4.14
- net P1.6: no longer J4.10
- net P1.7: no longer J4.8
- net P2.3: no longer J4.6
- net P2.6: no longer J4.2
- net P5.0: no longer J4.1
- net P5.1: no longer J4.3
- net P5.2: no longer J4.5
- net P5.3: no longer J4.7
- net P5.4: no longer J4.9
- net P5.6: no longer J4.11
- net P5.7: no longer J4.13
- net P6.0: no longer J4.15
- net P6.1: no longer J4.17
- net P6.2: no longer J4.19
- net P6.3: no longer J4.21
- net P6.4: no longer J4.23
- net P6.5: no longer J4.24
- net P6.6: no longer J4.22
- net P6.7: no longer J4.20
