File: nest_interface/eagle/rev_b/nest_interface_b.brd (EAGLE design)
At the start: 133.3 x 110.5 mm, 141 parts, among them J1 MOLEX_MICRO_USB_B_047346, J10 CONN_BLOCK_2, J11 CONN_BLOCK_2, J12 CONN_BLOCK_2, J13 CONN_BLOCK_2, J14 CONN_BLOCK_3, J15 CONN_BLOCK_3, J16 CONN_BLOCK_7, J17 CONN_BLOCK_7, J18 CONN_BLOCK_8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

Commit message: moved gpio interrupt to pin2.7
Parts:
- added TP13, TP14: TEST_POINT_0.040IN, nest_interface:TESTPOINT_0.040IN
Connections:
- removed net EPIC_P2.7: J3.3, U1.P$53
- new net EPIC_P1.2: J3.3, U1.P$30
- net 5.6V_SUPPLY: now also TP13.TESTPOINT
- net GND: now also TP14.TESTPOINT
- net TSTAT_IN_I2C_INT: now also U1.P$53; no longer U1.P$30
Routing:
- net EPIC_P2.7: track 33.4 -> 0.00 mm, vias 1 -> 0
- net TSTAT_IN_I2C_INT: track 79.5 -> 110.0 mm, vias 4 -> 5
- net N$9: track 24.2 -> 3.80 mm
- net N$12: track 19.9 -> 2.60 mm
- net 5.6V_SUPPLY: track 33.9 -> 39.8 mm
Other:
- board text added: "2012/11/27"
- board text removed: "2012/10/20"
Changed lines of the file:
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@@
 <text x="4.064" y="56.388" size="1.016" layer="21" font="vector" ratio="12" align="bottom-center">NEST</text>
 <text x="93.98" y="83.439" size="2.032" layer="21" font="vector" ratio="15">NEST Interface Board</text>
-<text x="93.98" y="81.28" size="1.016" layer="21" font="vector" ratio="12">2012/10/20</text>
+<text x="93.98" y="81.28" size="1.016" layer="21" font="vector" ratio="12">2012/11/27</text>
 <text x="58.928" y="3.302" size="1.016" layer="21" font="vector" ratio="12" rot="R270" align="center-left">TX</text>
 <text x="61.722" y="3.302" size="1.016" layer="21" font="vector" ratio="12" rot="R270" align="center-left">RX</text>
@@
 <text x="25.4" y="81.788" size="1.016" layer="21" font="vector" ratio="12" rot="R90">24VAC SIGNALS</text>
 <hole x="87.63" y="64.77" drill="3.175"/>
+<text x="128.016" y="94.488" size="1.016" layer="21" font="vector" ratio="12" align="center-right">5.6V</text>
+<text x="128.016" y="91.44" size="1.016" layer="21" font="vector" ratio="12" align="center-right">GND</text>
+<text x="44.577" y="4.064" size="1.016" layer="21" font="vector" ratio="12" align="bottom-center">3V</text>
+<text x="48.387" y="4.064" size="1.016" layer="21" font="vector" ratio="12" align="bottom-center">GND</text>
 </plain>
 <attributes>
@@
 <attribute name="VALUE" x="86.487" y="53.721" size="1.016" layer="27" font="vector" ratio="12" rot="R270"/>
 </element>
-<element name="TP1" library="nest_interface" package="TESTPOINT_0.040IN" value="TEST_POINT_0.040IN" x="44.577" y="2.54">
+<element name="TP1" library="nest_interface" package="TESTPOINT_0.040IN" value="TEST_POINT_0.040IN" x="44.577" y="2.54" smashed="yes">
 <attribute name="DIGIKEY" value="5001K-ND" x="44.577" y="2.54" size="1.778" layer="27" font="vector" ratio="12" display="off"/>
+<attribute name="VALUE" x="44.577" y="0" size="1.016" layer="27" font="vector" ratio="12" align="bottom-center"/>
 </element>
-<element name="TP2" library="nest_interface" package="TESTPOINT_0.040IN" value="TEST_POINT_0.040IN" x="48.387" y="2.54">
+<element name="TP2" library="nest_interface" package="TESTPOINT_0.040IN" value="TEST_POINT_0.040IN" x="48.387" y="2.54" smashed="yes">
 <attribute name="DIGIKEY" value="5001K-ND" x="48.387" y="2.54" size="1.778" layer="27" font="vector" ratio="12" display="off"/>
+<attribute name="VALUE" x="48.387" y="0" size="1.016" layer="27" font="vector" ratio="12" align="bottom-center"/>
 </element>
 <element name="TP3" library="nest_interface" package="TESTPOINT_0.040IN" value="TEST_POINT_0.040IN" x="86.741" y="35.306">
@@
 <attribute name="VALUE" x="78.74" y="10.287" size="1.27" layer="27"/>
 </element>
+<element name="TP13" library="nest_interface" package="TESTPOINT_0.040IN" value="TEST_POINT_0.040IN" x="129.54" y="94.488" smashed="yes">
+<attribute name="DIGIKEY" value="5001K-ND" x="129.54" y="94.488" size="0.254" layer="27" font="vector" ratio="12" display="off"/>
+<attribute name="TITLE" value="Nest Interface Board" x="129.54" y="94.488" size="1.778" layer="27" display="off"/>
+<attribute name="REV" value="A" x="129.54" y="94.488" size="1.778" layer="27" display="off"/>
+<attribute name="VALUE" x="129.54" y="91.948" size="1.016" layer="27" font="vector" ratio="12" align="bottom-center"/>
+</element>
+<element name="TP14" library="nest_interface" package="TESTPOINT_0.040IN" value="TEST_POINT_0.040IN" x="129.54" y="91.44" smashed="yes">
+<attribute name="DIGIKEY" value="5001K-ND" x="129.54" y="91.44" size="0.254" layer="27" font="vector" ratio="12" display="off"/>
+<attribute name="TITLE" value="Nest Interface Board" x="129.54" y="91.44" size="1.778" layer="27" display="off"/>
+<attribute name="REV" value="A" x="129.54" y="91.44" size="1.778" layer="27" display="off"/>
+<attribute name="VALUE" x="129.54" y="88.9" size="1.016" layer="27" font="vector" ratio="12" align="bottom-center"/>
+</element>
 </elements>
 <signals>
@@
 <wire x1="119.192" y1="13.8" x2="118.237" y2="14.755" width="0.254" layer="1"/>
 <wire x1="118.237" y1="14.755" x2="118.237" y2="15.113" width="0.254" layer="1"/>
+<contactref element="TP14" pad="TESTPOINT"/>
 </signal>
 <signal name="N$1">
@@
 <wire x1="64.355" y1="12.885" x2="63.246" y2="12.885" width="0.254" layer="1"/>
 <via x="63.246" y="12.885" extent="1-16" drill="0.4064"/>
-<wire x1="67.31" y1="32.385" x2="67.31" y2="30.607" width="0.254" layer="1"/>
-<wire x1="67.31" y1="30.607" x2="66.802" y2="30.099" width="0.254" layer="1"/>
-<wire x1="66.802" y1="30.099" x2="65.786" y2="30.099" width="0.254" layer="1"/>
-<wire x1="65.786" y1="30.099" x2="65.151" y2="30.734" width="0.254" layer="1"/>
-<via x="65.151" y="30.734" extent="1-16" drill="0.4064"/>
-<wire x1="65.151" y1="30.734" x2="65.151" y2="14.79" width="0.254" layer="16"/>
+<wire x1="67.31" y1="32.385" x2="67.31" y2="30.607" width="0" layer="19" extent="1-16"/>
+<wire x1="67.31" y1="30.607" x2="66.802" y2="30.099" width="0" layer="19" extent="1-16"/>
+<wire x1="66.802" y1="30.099" x2="65.786" y2="30.099" width="0" layer="19" extent="1-16"/>
+<wire x1="65.786" y1="30.099" x2="62.738" y2="28.321" width="0" layer="19" extent="1-16"/>
+<via x="62.738" y="28.321" extent="1-16" drill="0.4064"/>
+<wire x1="62.738" y1="28.321" x2="65.151" y2="14.79" width="0" layer="19" extent="1-16"/>
 <wire x1="65.151" y1="14.79" x2="63.246" y2="12.885" width="0.254" layer="16"/>
 </signal>
@@
 <wire x1="66.955" y1="12.885" x2="66.955" y2="14.732" width="0.254" layer="1"/>
 <via x="66.955" y="14.732" extent="1-16" drill="0.4064"/>
-<wire x1="66.04" y1="32.385" x2="66.04" y2="31.242" width="0.254" layer="1"/>
-<wire x1="66.04" y1="31.242" x2="66.421" y2="30.861" width="0.254" layer="1"/>
-<via x="66.421" y="30.861" extent="1-16" drill="0.4064"/>
-<wire x1="66.421" y1="30.861" x2="66.421" y2="15.266" width="0.254" layer="16"/>
+<wire x1="66.04" y1="32.385" x2="66.04" y2="31.242" width="0" layer="19" extent="1-16"/>
+<wire x1="66.04" y1="31.242" x2="62.738" y2="29.591" width="0" layer="19" extent="1-16"/>
+<via x="62.738" y="29.591" extent="1-16" drill="0.4064"/>
+<wire x1="62.738" y1="29.591" x2="66.421" y2="15.266" width="0" layer="19" extent="1-16"/>
 <wire x1="66.421" y1="15.266" x2="66.955" y2="14.732" width="0.254" layer="16"/>
 </signal>
@@
 <wire x1="58.42" y1="35.56" x2="58.42" y2="54.61" width="0.254" layer="1"/>
 </signal>
-<signal name="EPIC_P2.7">
-<contactref element="U1" pad="P$53"/>
-<contactref element="J3" pad="3"/>
-<via x="57.15" y="54.61" extent="1-16" drill="0.4064"/>
-<wire x1="55.88" y1="32.385" x2="55.88" y2="34.036" width="0.254" layer="1"/>
-<wire x1="55.88" y1="34.036" x2="57.15" y2="35.306" width="0.254" layer="1"/>
-<wire x1="57.15" y1="35.306" x2="57.15" y2="54.61" width="0.254" layer="1"/>
-<wire x1="57.15" y1="54.61" x2="57.15" y2="63.5" width="0.254" layer="16"/>
-<wire x1="57.15" y1="63.5" x2="55.88" y2="64.77" width="0.254" layer="16"/>
-</signal>
 <signal name="#KEYPAD_ENABLE">
 <contactref element="U1" pad="P$4"/>
@@
 <contactref element="U7" pad="14"/>
 <contactref element="R24" pad="2"/>
-<contactref element="U1" pad="P$30"/>
 <wire x1="78.74" y1="54.356" x2="74.93" y2="54.356" width="0.254" layer="16"/>
 <via x="74.93" y="54.356" extent="1-16" drill="0.4064" diameter="0.4064"/>
 <wire x1="74.93" y1="54.356" x2="60.706" y2="54.356" width="0.254" layer="1"/>
 <wire x1="60.706" y1="54.356" x2="59.69" y2="55.372" width="0.254" layer="1"/>
-<wire x1="59.69" y1="55.372" x2="59.69" y2="56.515" width="0.254" layer="1"/>
 <wire x1="78.74" y1="54.356" x2="84.074" y2="49.022" width="0.254" layer="16"/>
 <wire x1="84.074" y1="49.022" x2="84.074" y2="42.799" width="0.254" layer="16"/>
@@
 <wire x1="86.741" y1="35.306" x2="86.741" y2="33.274" width="0.254" layer="1"/>
 <wire x1="86.741" y1="33.274" x2="85.852" y2="32.385" width="0.254" layer="1"/>
+<contactref element="U1" pad="P$53"/>
+<via x="57.15" y="54.61" extent="1-16" drill="0.4064"/>
+<wire x1="55.88" y1="32.385" x2="55.88" y2="34.036" width="0.254" layer="1"/>
+<wire x1="55.88" y1="34.036" x2="57.15" y2="35.306" width="0.254" layer="1"/>
+<wire x1="57.15" y1="35.306" x2="57.15" y2="54.61" width="0.254" layer="1"/>
+<wire x1="57.15" y1="54.61" x2="57.15" y2="63.5" width="0.254" layer="16"/>
+<wire x1="57.15" y1="54.61" x2="59.69" y2="55.372" width="0" layer="19" extent="1-16"/>
 </signal>
 <signal name="TSTAT_IN_I2C_RST">
@@
 <wire x1="121.16" y1="94.474" x2="123.684" y2="94.474" width="0.6096" layer="1"/>
 <wire x1="123.684" y1="94.474" x2="129.54" y2="100.33" width="0.6096" layer="1"/>
+<contactref element="TP13" pad="TESTPOINT"/>
+<wire x1="129.54" y1="94.488" x2="123.684" y2="94.474" width="0.6096" layer="1"/>
 </signal>
 <signal name="LCDP_STE1">
@@
 <wire x1="48.224" y1="90.206" x2="47.625" y2="90.805" width="0.254" layer="1"/>
 </signal>
+<signal name="EPIC_P1.2">
+<contactref element="U1" pad="P$30"/>
+<contactref element="J3" pad="3"/>
+<wire x1="59.69" y1="56.515" x2="55.88" y2="64.77" width="0" layer="19" extent="1-1"/>
+</signal>
 </signals>

Commit message: fuck fuck fuck
Routing:
- net TSTAT_IN_I2C_INT: track 110.0 -> 66.9 mm, vias 5 -> 4
- net N$12: track 2.60 -> 23.4 mm
- net N$9: track 3.80 -> 23.8 mm
- net #KEYPAD_ENABLE: track 104.3 -> 114.7 mm
- net EPIC_P1.2: track 0.00 -> 9.83 mm
- net GND: track 246.3 -> 254.2 mm
- net VCC: track 595.7 -> 600.0 mm
- net TSTAT2_UP_OUT: track 19.7 -> 22.1 mm
- net TSTAT2_HELP_OUT: track 19.7 -> 22.1 mm
- net TSTAT2_ENTER_OUT: track 20.0 -> 22.3 mm
- net TSTAT2_DOWN_OUT: track 19.7 -> 22.1 mm
- net TSTAT1_UP_OUT: track 16.9 -> 19.3 mm
- net TSTAT1_ON/OFF_OUT: track 16.9 -> 19.3 mm
- net TSTAT1_MENU_OUT: track 16.9 -> 19.3 mm
- net TSTAT1_HELP_OUT: track 17.0 -> 19.3 mm
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